File: board/fabpidex.kicad_pcb (KiCad board)
At the start: 2 copper layers, 10 x 25.4 mm, 28 parts, among them J1 USB_C_Receptacle, J2 Vdrive, J3 GND, M1 MountingHole_2.2mm_M2_Pad_Via, M2 MountingHole_2.2mm_M2_Pad_Via, Q1 SSM6J507NU, Q2 Q_Photo_NPN, U1 STUSB4500, U2 MCP1799T-3302H_TT, U3 ATtiny816-M

Commit message: Fix up issues
Routing:
- net GND: track 12.0 -> 18.6 mm, vias 3 -> 5
- net VBUS: track 15.3 -> 17.2 mm, vias 3 -> 4
Other:
- board text added: "5-20v"
- board text added: "GND"
- board text added: "fabpidex v1.1"
