File: board/fabpidex.kicad_pcb (KiCad board)
At the start: 2 copper layers, 10 x 25.4 mm, 28 parts, among them J1 USB_C_Receptacle, J2 Vdrive, J3 GND, M1 MountingHole_2.2mm_M2_Pad_Via, M2 MountingHole_2.2mm_M2_Pad_Via, Q1 SSM6J507NU, Q2 Q_Photo_NPN, U1 STUSB4500, U2 MCP1799T-3302H_TT, U3 ATtiny816-M

Commit message: Fix up issues
Routing:
- net GND: track 12.0 -> 18.6 mm, vias 3 -> 4
- net VBUS: track 15.3 -> 17.2 mm, vias 3 -> 4
Other:
- board text added: "5-20v"
- board text added: "GND"
- board text added: "fabpidex v1.1"

Commit message: Minor cosmetics
Other:
- board text added: "fpx.oxplot.com"
Changed lines of the file:
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@@
   (general
     (thickness 1.6)
-    (drawings 15)
+    (drawings 23)
     (tracks 182)
     (zones 0)
@@
     (34 B.Paste user)
     (35 F.Paste user)
-    (36 B.SilkS user hide)
+    (36 B.SilkS user)
     (37 F.SilkS user)
     (38 B.Mask user)
@@
   (module fabpidex:USB4105-GF-A (layer F.Cu)
     (at 160.8328 92.4306 270)
-    (fp_text reference J1 (at 5.6896 1.6002 180) (layer F.SilkS)
+    (fp_text reference J1 (at 0.5294 -4.8472 270) (layer F.SilkS)
       (effects (font (size 0.6 0.6) (thickness 0.127)))
     )
@@
     )
   )
+  (gr_text fpx.oxplot.com (at 161.16 98.03) (layer F.SilkS)
+    (effects (font (size 0.5 0.5) (thickness 0.125)))
+  )
+  (gr_line (start 166.24 103.84) (end 166.24 103.26) (layer B.SilkS) (width 0.127))
+  (gr_line (start 164.97 103.84) (end 166.24 103.84) (layer B.SilkS) (width 0.127))
+  (gr_line (start 164.75 103.62) (end 164.97 103.84) (layer B.SilkS) (width 0.127))
+  (gr_text 5-20v (at 164.51 102.15 90) (layer B.SilkS)
+    (effects (font (size 0.6 0.6) (thickness 0.127)) (justify mirror))
+  )
+  (gr_line (start 164.76 84.04) (end 164.76 84.28) (layer B.SilkS) (width 0.127))
+  (gr_line (start 165.16 83.64) (end 164.76 84.04) (layer B.SilkS) (width 0.127))
+  (gr_text GND (at 164.61 84.95) (layer B.SilkS)
+    (effects (font (size 0.7 0.7) (thickness 0.175)) (justify mirror))
+  )
   (gr_text "fabpidex\nv1.1" (at 160.43 86.27) (layer F.SilkS)

Commit message: More cosmetics
Parts:
- moved ? 0.41 mm to (159.1, 99.8)
Other:
- board text added: "fabpidex v1.3"
- board text removed: "fabpidex v1.1"
Changed lines of the file:
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@@
   )
   (module Fiducial:Fiducial_0.5mm_Mask1mm (layer F.Cu)
-    (at 159.35 99.48)
+    (at 159.11 99.81)
     (descr "Circular Fiducial, 0.5mm bare copper, 1mm soldermask opening (Level C)")
     (tags fiducial)
@@
     )
   )
-  (gr_text fpx.oxplot.com (at 161.16 98.03) (layer F.SilkS)
+  (gr_text fpx.oxplot.com (at 161.49 98.62) (layer F.SilkS)
     (effects (font (size 0.5 0.5) (thickness 0.125)))
   )
@@
     (effects (font (size 0.7 0.7) (thickness 0.175)) (justify mirror))
   )
-  (gr_text "fabpidex\nv1.1" (at 160.43 86.27) (layer F.SilkS)
-    (effects (font (size 0.6 0.6) (thickness 0.127)))
+  (gr_text "fabpidex\nv1.3" (at 160.43 86.27) (layer F.SilkS)
+    (effects (font (size 0.5 0.5) (thickness 0.125)))
   )
   (gr_line (start 164.6 99.36) (end 165.68 100.44) (layer F.SilkS) (width 0.127))
